File: schema/optics_r001.sch (EAGLE design)
At the start: 28 parts, among them Q1 Si2333DDS, Q2 Si2342DS, U1 OPA2380, U2 OPA2380, U3 iC-HKB, X1 MAIN_CON, X2 MikroBus_3, X3 PWM_1, X4 PWM_2

Commit message: finialzing optics_r001 before sending to fab
Parts:
- added DS4: LSR, diode:LED/YELLOW/1206/KINGBRIGHT
- added DS5: ID1, diode:LED/BLUE/1206/KINGBRIGHT
- added DS6: ID2, diode:LED/RED/1206/KINGBRIGHT
- added DS7: ID3, diode:LED/BLUE/1206/KINGBRIGHT
- added DS8: ID4, diode:LED/YELLOW/1206/KINGBRIGHT
- added DS9: (no value), diode:LED/BLUE/TH/5MM/CREE
- added MH1: MTG_HOLE/M3/PLATED, mechanical:MTG_HOLE/M3/PLATED
- added MH2, MH3: MTG_HOLE/M2/PLATED, mechanical:MTG_HOLE/M2/PLATED
- added MP1: (no value), mechanical:LENS_HOLDER/M9/LOW-PROFILE
- added R10, R12: 80.6, rcl:R/1%/0805/0.125W
- added R11, R13: 150, rcl:R/1%/0805/0.125W
- added R9: 137, rcl:R/1%/0805/0.125W
- added TP1, TP2, TP3: (no value), pad:TP/RECT_5X2.5
- added TP10, TP5, TP6: (no value), pad:TP/CIRCLE_1.5
- added TP7, TP8: (no value), pad:TP/OVAL_3X1.5
- added TP9: (no value), pad:TP/CIRCLE_2
- added X5: TILT_SERVO, io:HEADER-1X03/MALE/100MIL/TH/BREAKAWAY
- C1: device rcl:C/0805/10V -> rcl:C/10%/0805/10V
- C2: value 100n -> 0.1u; device rcl:C/0805/10V -> rcl:C/5%/0805/10V
- C3: device rcl:C/0805/10V -> rcl:C/1%/0805/10V
- C4: device rcl:C/0805/10V -> rcl:C/5%/0805/10V
- D1: value PL_450B -> (none)
- DS1: value +5V -> P5V; device diode:LED/1206/YELLOW -> diode:LED/YELLOW/1206/KINGBRIGHT
- DS2: value +3.3V -> P3_3V; device diode:LED/1206/YELLOW -> diode:LED/YELLOW/1206/KINGBRIGHT
- DS3: device diode:LED/1206/ORANGE -> diode:LED/RED/1206/KINGBRIGHT
- Q1: value Si2333DDS -> (none); device transistor:MOSFET_P-TYPE -> transistor:MOSFET_P-TYPE/SI2333DDS
- Q2: value Si2342DS -> (none); device transistor:MOSFET_N-TYPE -> transistor:MOSFET_N-TYPE/SI2342DS
- R1, R2, R5, RK1, RK2: device rcl:R/0805/0.125W -> rcl:R/1%/0805/0.125W
- R3: value 0.92 -> 0.82; device rcl:R_SENSE/1206/0.25W -> rcl:R_SENSE/1%/1206/0.5W
- R4: device rcl:R_POT/10K -> rcl:R_POT/T93YB; MPN (none) -> T93YB103KT20
- R6: value 137 -> 150; device rcl:R/0805/0.125W -> rcl:R/1%/0805/0.125W
- R7, R8: value 56 -> 68; device rcl:R/0805/0.125W -> rcl:R/1%/0805/0.125W
- U1, U2: value OPA2380 -> (none)
- U3: device ic:IC-HK/B -> ic:IC-HKB
- X1: value MAIN_CON -> (none); device io:HEADER-2X10MALE/100MIL/TH/SHROUDED -> io:HEADER-1X10/MALE/100MIL/TH/BREAKAWAY
- X2: value MikroBus_3 -> (none); device io:MIKROE_BUS_CONN/FEMALE/100MIL/TH -> io:HEADER-1X10/MALE/100MIL/TH/BREAKAWAY
- X3: value PWM_1 -> MikroBus_3; device io:HEADER-1X03/MALE/100MIL/TH/BREAKAWAY -> io:MIKROE_BUS_CONN/SOCKET/NO_OUTLINE/COMPACT
- X4: value PWM_2 -> PAN_SERVO
Connections:
- net N$1 renamed RX_OPAMP_OUT4
- net N$10 renamed RX_OPAMP_OUT2
- net N$15 renamed RX_OPAMP_OUT3
- net N$5 renamed RX_OPAMP_OUT1
- removed net +5V_LSR: C1.1, C2.1, C3.1, D1.A, Q1.D, U3.VDD
- new net LED_5V_LSR_ANODE: DS4.A, R9.2
- new net LED_ID1_ANODE: DS5.A, R10.2
- new net LED_ID2_ANODE: DS6.A, R11.2
- new net LED_ID3_ANODE: DS7.A, R12.2
- new net LED_ID4_ANODE: DS8.A, R13.2
- new net P5V_LSR: C1.1, C2.1, C3.1, D1.A, DS9.A, Q1.D, R9.1, TP2.1, U3.VDD
- net GND: now also DS4.C, DS5.C, DS6.C, DS7.C, DS8.C, MH1.1, MH2.1, MH3.1, MP1.P$1, MP1.P$2, X1.10, X3.GND1, X3.GND2, X5.3; no longer X1.20, X2.GND1, X2.GND2, X3.3
- net IN: now also TP1.1
- net LSR_ENB: now also TP9.1, X2.8; no longer X1.5
- net LSR_EN_CH1: now also TP7.1, X2.9; no longer X1.7
- net LSR_EN_CH2: now also TP8.1, X2.10; no longer X1.9
- net LSR_ILIM_VSENSE: now also TP10.1, X1.3; no longer X1.6
- net LSR_ISENSE_LS_N: now also TP6.1, X1.5; no longer X1.10
- net LSR_ISENSE_LS_P: now also DS9.C, TP5.1, X1.4; no longer X1.8
- net OPAMP_OUT: now also TP2.1
- net OUT: now also TP3.1
- net P3_3V: now also TP3.1, X2.1, X3.3V3; no longer X1.2, X2.3V3
- net P5V: now also R10.1, R11.1, R12.1, R13.1, TP1.1, X3.5V, X5.2; no longer X2.5V, X3.2
- net RB1_MB2_CS: now also X2.4, X3.CS; no longer X1.11, X2.CS
- net RD0_PWM1: now also X1.2, X4.1; no longer X1.3, X3.1
- net RD3_PWM4: now also X2.2, X5.1; no longer X1.4, X4.1
- net RE9_MB2_INT2: now also X2.3, X3.INT; no longer X1.19, X2.INT
- net RG6_SPI2_SCK: now also X2.5, X3.SCK; no longer X1.13, X2.SCK
- net RG7_SPI2_MISO: now also X2.6, X3.MISO; no longer X1.15, X2.MISO
- net RG8_SPI2_MOSI: now also X2.7, X3.MOSI; no longer X1.17, X2.MOSI
- net RX_AMP1_OUT: now also X1.6; no longer X1.12
- net RX_AMP2_OUT: now also X1.7; no longer X1.14
- net RX_AMP3_OUT: now also X1.8; no longer X1.16
- net RX_AMP4_OUT: now also X1.9; no longer X1.18
Other:
- note added: "10bit A/D (Vref=3.3V) res=3.22mV/bit Isense res=3.9mA/bit"
- note added: "I=20mA w/ V_f=2V"
- note added: "I=20mA w/ V_f=3.3V"
- note added: "I~=20mA w/ V_f=2V"
- note added: "I~=20mA w/ V_f~=2V"
- note added: "OPA2380"
- note added: "resistor used to slow turn on of pass transistor by 5us (not full-blow slow start circuit)"
- note removed: "10bit A/D (Vref=3.3V) res=3.22mV/bit Isense res=3.5mA/bit"
- note removed: "I=20mA w/ V_f~=2.18V"
- note removed: "I=21mA w/ V_f=2.3V"
- note removed: "OPA380"
- note removed: "text R used to slow turn on of pass transistor by 5us (not full-blow slow start circuit)"
- moved on the sheet: C1, C2, C3, C4, D2, R4, R5, U1_A, U1_B, U2_A, U2_B, X4

Commit message: general file cleanup
Parts:
- DS2, DS4, DS9, R7, R9: DNI (none) -> DNI
Changed lines of the file:
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@@
 <part name="GND10" library="misc" deviceset="GND" device=""/>
 <part name="GND11" library="misc" deviceset="GND" device=""/>
-<part name="R7" library="rcl" deviceset="R" device="/0805/0.125W" technology="/1%" value="68"/>
-<part name="DS2" library="diode" deviceset="LED" device="/1206/KINGBRIGHT" technology="/YELLOW" value="P3_3V"/>
+<part name="R7" library="rcl" deviceset="R" device="/0805/0.125W" technology="/1%" value="68">
+<attribute name="DNI" value="DNI"/>
+</part>
+<part name="DS2" library="diode" deviceset="LED" device="/1206/KINGBRIGHT" technology="/YELLOW" value="P3_3V">
+<attribute name="DNI" value="DNI"/>
+</part>
 <part name="R8" library="rcl" deviceset="R" device="/0805/0.125W" technology="/1%" value="68"/>
 <part name="DS3" library="diode" deviceset="LED" device="/1206/KINGBRIGHT" technology="/RED" value="LSR_ENB"/>
@@
 <part name="MP1" library="mechanical" deviceset="LENS_HOLDER" device="/M9/LOW-PROFILE"/>
 <part name="GND30" library="misc" deviceset="GND" device=""/>
-<part name="R9" library="rcl" deviceset="R" device="/0805/0.125W" technology="/1%" value="137"/>
-<part name="DS4" library="diode" deviceset="LED" device="/1206/KINGBRIGHT" technology="/YELLOW" value="LSR"/>
+<part name="R9" library="rcl" deviceset="R" device="/0805/0.125W" technology="/1%" value="137">
+<attribute name="DNI" value="DNI"/>
+</part>
+<part name="DS4" library="diode" deviceset="LED" device="/1206/KINGBRIGHT" technology="/YELLOW" value="LSR">
+<attribute name="DNI" value="DNI"/>
+</part>
 <part name="GND29" library="misc" deviceset="GND" device=""/>
 <part name="R10" library="rcl" deviceset="R" device="/0805/0.125W" technology="/1%" value="80.6"/>
@@
 <part name="P+9" library="misc" deviceset="P3_3V" device=""/>
 <part name="DS9" library="diode" deviceset="LED" device="/TH/5MM/CREE" technology="/BLUE">
+<attribute name="DNI" value="DNI"/>
 <attribute name="EAGLEUP" value="LED5MM_GREEN;;DNI"/>
 </part>
@@
 <text x="-45" y="9" size="1" layer="97" ratio="12">I~=20mA w/
 V_f=2V</text>
-<text x="-25" y="-34" size="1" layer="97" ratio="12">I=20mA w/
+<text x="-25" y="-33" size="1" layer="97" ratio="12">I=20mA w/
 V_f=2V</text>
 <text x="-25" y="9" size="1" layer="97" ratio="12">I~=20mA w/
@@
 </instance>
 <instance part="Q2" gate="G$1" x="1" y="-21">
-<attribute name="MPN" x="1" y="-21" size="1" layer="96" ratio="12"/>
+<attribute name="MPN" x="4" y="-22.5" size="1" layer="96" ratio="12"/>
 </instance>
 <instance part="D1" gate="G$1" x="76" y="11">
@@
 <instance part="GND10" gate="GND" x="-29" y="-56"/>
 <instance part="GND11" gate="GND" x="-29" y="-11"/>
-<instance part="R7" gate="G$1" x="-49" y="11" rot="MR270"/>
-<instance part="DS2" gate="G$1" x="-49" y="-4"/>
+<instance part="R7" gate="G$1" x="-49" y="11" rot="MR270">
+<attribute name="DNI" x="-52.5" y="12" size="1" layer="96" ratio="12" rot="MR270" display="name"/>
+</instance>
+<instance part="DS2" gate="G$1" x="-49" y="-4">
+<attribute name="DNI" x="-47" y="-7" size="1" layer="96" ratio="12" display="name"/>
+</instance>
 <instance part="R8" gate="G$1" x="-29" y="-31" rot="MR270"/>
 <instance part="DS3" gate="G$1" x="-29" y="-48"/>
@@
 </instance>
 <instance part="GND30" gate="GND" x="61" y="8"/>
-<instance part="R9" gate="G$1" x="31" y="11" rot="MR270"/>
-<instance part="DS4" gate="G$1" x="31" y="-4"/>
+<instance part="R9" gate="G$1" x="31" y="11" rot="MR270">
+<attribute name="DNI" x="26.5" y="9.5" size="1" layer="96" ratio="12" rot="MR90" display="name"/>
+</instance>
+<instance part="DS4" gate="G$1" x="31" y="-4">
+<attribute name="DNI" x="33" y="-7" size="1" layer="96" ratio="12" display="name"/>
+</instance>
 <instance part="GND29" gate="GND" x="31" y="-11"/>
 <instance part="R10" gate="G$1" x="166" y="-98" rot="MR270"/>
@@
 <instance part="P+6" gate="+5V" x="75" y="-98"/>
 <instance part="P+9" gate="G$1" x="52" y="-98"/>
-<instance part="DS9" gate="G$1" x="91" y="11"/>
+<instance part="DS9" gate="G$1" x="91" y="11">
+<attribute name="DNI" x="93" y="9.5" size="1" layer="96" ratio="12" display="name"/>
+</instance>
 <instance part="FRAME1" gate="G$2" x="217" y="-192"/>
 <instance part="FRAME1" gate="G$1" x="-122.09" y="-192"/>
