File: schema/optics_r002/optics_r002.sch (EAGLE design)
At the start: 53 parts, among them U3 iC-HKB, X3 MikroBus_3, X4 PAN_SERVO, X5 TILT_SERVO

Commit message: updated reworks 1-4 to schematic r002
Parts:
- added C5, C6: 4700u, rcl:C_POL/20%/RADIAL/25V/16X35
- added C7, C8: 0.1u, rcl:C/5%/0805/10V
- added X6: REWORK, io:HEADER-1X03/MALE/100MIL/TH/BREAKAWAY
Connections:
- new net GND_A: X6.2
- new net P12V: D2.C, X6.1
- net GND: now also C5.2, C6.2, C7.2, C8.2, X6.3
- net P5V: now also C5.1, C6.1, C7.1, C8.1; no longer D2.C
Other:
- moved on the sheet: X1, X2, X4, X5

Commit message: revision 1 uploaded and sent for review
Other:
- note added: "resistor used to slow turn on of pass transistor by 5us (not full-blown slow start circuit)"
- note removed: "resistor used to slow turn on of pass transistor by 5us (not full-blow slow start circuit)"
- moved on the sheet: C4, TP10
Changed lines of the file:
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@@
 <grid distance="1" unitdist="mm" unit="mm" style="lines" multiple="1" display="yes" altdistance="0.5" altunitdist="mm" altunit="mm"/>
 <layers>
-<layer number="1" name="Top" color="1" fill="1" visible="yes" active="no"/>
-<layer number="16" name="Bottom" color="12" fill="1" visible="yes" active="no"/>
-<layer number="17" name="Pads" color="2" fill="1" visible="yes" active="no"/>
-<layer number="18" name="Vias" color="2" fill="1" visible="yes" active="no"/>
-<layer number="19" name="Unrouted" color="6" fill="1" visible="yes" active="no"/>
-<layer number="20" name="Dimension" color="15" fill="1" visible="yes" active="no"/>
-<layer number="21" name="tPlace" color="25" fill="1" visible="yes" active="no"/>
-<layer number="22" name="bPlace" color="7" fill="1" visible="yes" active="no"/>
-<layer number="23" name="tOrigins" color="15" fill="1" visible="yes" active="no"/>
-<layer number="24" name="bOrigins" color="15" fill="1" visible="yes" active="no"/>
-<layer number="25" name="tNames" color="7" fill="1" visible="yes" active="no"/>
-<layer number="26" name="bNames" color="7" fill="1" visible="yes" active="no"/>
-<layer number="27" name="tValues" color="7" fill="1" visible="yes" active="no"/>
-<layer number="28" name="bValues" color="7" fill="1" visible="yes" active="no"/>
+<layer number="1" name="Top" color="1" fill="1" visible="no" active="no"/>
+<layer number="16" name="Bottom" color="12" fill="1" visible="no" active="no"/>
+<layer number="17" name="Pads" color="2" fill="1" visible="no" active="no"/>
+<layer number="18" name="Vias" color="2" fill="1" visible="no" active="no"/>
+<layer number="19" name="Unrouted" color="6" fill="1" visible="no" active="no"/>
+<layer number="20" name="Dimension" color="15" fill="1" visible="no" active="no"/>
+<layer number="21" name="tPlace" color="25" fill="1" visible="no" active="no"/>
+<layer number="22" name="bPlace" color="7" fill="1" visible="no" active="no"/>
+<layer number="23" name="tOrigins" color="15" fill="1" visible="no" active="no"/>
+<layer number="24" name="bOrigins" color="15" fill="1" visible="no" active="no"/>
+<layer number="25" name="tNames" color="7" fill="1" visible="no" active="no"/>
+<layer number="26" name="bNames" color="7" fill="1" visible="no" active="no"/>
+<layer number="27" name="tValues" color="7" fill="1" visible="no" active="no"/>
+<layer number="28" name="bValues" color="7" fill="1" visible="no" active="no"/>
 <layer number="29" name="tStop" color="7" fill="3" visible="no" active="no"/>
 <layer number="30" name="bStop" color="15" fill="6" visible="no" active="no"/>
@@
 <layer number="35" name="tGlue" color="7" fill="4" visible="no" active="no"/>
 <layer number="36" name="bGlue" color="7" fill="5" visible="no" active="no"/>
-<layer number="37" name="tTest" color="7" fill="1" visible="yes" active="no"/>
-<layer number="38" name="bTest" color="7" fill="1" visible="yes" active="no"/>
+<layer number="37" name="tTest" color="7" fill="1" visible="no" active="no"/>
+<layer number="38" name="bTest" color="7" fill="1" visible="no" active="no"/>
 <layer number="39" name="tKeepout" color="4" fill="11" visible="no" active="no"/>
 <layer number="40" name="bKeepout" color="1" fill="11" visible="no" active="no"/>
@@
 <layer number="44" name="Drills" color="7" fill="1" visible="no" active="no"/>
 <layer number="45" name="Holes" color="7" fill="1" visible="no" active="no"/>
-<layer number="46" name="Milling" color="3" fill="1" visible="yes" active="no"/>
-<layer number="47" name="Measures" color="7" fill="1" visible="yes" active="no"/>
-<layer number="48" name="Document" color="7" fill="1" visible="yes" active="no"/>
-<layer number="49" name="Reference" color="7" fill="1" visible="yes" active="no"/>
-<layer number="50" name="dxf" color="7" fill="1" visible="yes" active="no"/>
-<layer number="51" name="tDocu" color="7" fill="1" visible="yes" active="no"/>
-<layer number="52" name="bDocu" color="7" fill="1" visible="yes" active="no"/>
-<layer number="53" name="tGND_GNDA" color="7" fill="9" visible="yes" active="no"/>
-<layer number="54" name="bGND_GNDA" color="1" fill="9" visible="yes" active="no"/>
-<layer number="56" name="wert" color="7" fill="1" visible="yes" active="no"/>
-<layer number="57" name="tCAD" color="7" fill="1" visible="yes" active="no"/>
+<layer number="46" name="Milling" color="3" fill="1" visible="no" active="no"/>
+<layer number="47" name="Measures" color="7" fill="1" visible="no" active="no"/>
+<layer number="48" name="Document" color="7" fill="1" visible="no" active="no"/>
+<layer number="49" name="Reference" color="7" fill="1" visible="no" active="no"/>
+<layer number="50" name="dxf" color="7" fill="1" visible="no" active="no"/>
+<layer number="51" name="tDocu" color="7" fill="1" visible="no" active="no"/>
+<layer number="52" name="bDocu" color="7" fill="1" visible="no" active="no"/>
+<layer number="53" name="tGND_GNDA" color="7" fill="9" visible="no" active="no"/>
+<layer number="54" name="bGND_GNDA" color="1" fill="9" visible="no" active="no"/>
+<layer number="56" name="wert" color="7" fill="1" visible="no" active="no"/>
+<layer number="57" name="tCAD" color="7" fill="1" visible="no" active="no"/>
 <layer number="90" name="Modules" color="5" fill="1" visible="yes" active="yes"/>
 <layer number="91" name="Nets" color="2" fill="1" visible="yes" active="yes"/>
@@
 <sheet>
 <plain>
-<text x="-18" y="-39" size="1" layer="97" ratio="12">1.06V &lt; Vref &lt; inf</text>
+<text x="-14" y="-38" size="1" layer="97" ratio="12">1.06V &lt; Vref &lt; inf</text>
 <text x="75" y="16" size="1" layer="97" ratio="12" rot="MR0">max 120mW/165mA
 typ 80mW/100mA</text>
@@
 <text x="5" y="-3" size="1" layer="97" ratio="12">resistor used to slow turn
 on of pass transistor by
-5us (not full-blow slow
+5us (not full-blown slow
 start circuit)</text>
 <text x="-45" y="9" size="1" layer="97" ratio="12">I~=20mA w/
@@
 <instance part="GND2" gate="GND" x="41" y="-62"/>
 <instance part="GND8" gate="GND" x="49" y="-62"/>
-<instance part="C4" gate="G$1" x="-1" y="-48" rot="MR270"/>
-<instance part="GND9" gate="GND" x="-1" y="-56"/>
+<instance part="C4" gate="G$1" x="1" y="-48" rot="MR270"/>
+<instance part="GND9" gate="GND" x="1" y="-56"/>
 <instance part="R6" gate="G$1" x="-29" y="11" rot="MR270"/>
 <instance part="DS1" gate="G$1" x="-29" y="-4"/>
@@
 <instance part="TP8" gate="G$1" x="20" y="-34" rot="R90"/>
 <instance part="TP9" gate="G$1" x="-19" y="-21" rot="R90"/>
-<instance part="TP10" gate="G$1" x="5" y="-42" rot="MR270"/>
+<instance part="TP10" gate="G$1" x="7" y="-42" rot="MR270"/>
 <instance part="GND28" gate="GND" x="127" y="-120"/>
 <instance part="MP1" gate="G$1" x="68" y="11">
@@
 <pinref part="C3" gate="G$1" pin="2"/>
 <wire x1="52" y1="-1" x2="52" y2="7" width="0.1524" layer="91"/>
-<label x="77" y="0" size="1" layer="95" ratio="12"/>
+<label x="77" y="-1" size="1" layer="95" ratio="12"/>
 <wire x1="76" y1="-1" x2="91" y2="-1" width="0.1524" layer="91"/>
 <wire x1="91" y1="-1" x2="106" y2="-1" width="0.1524" layer="91"/>
@@
 <segment>
 <pinref part="C4" gate="G$1" pin="2"/>
-<wire x1="-1" y1="-53" x2="-1" y2="-56" width="0.1524" layer="91"/>
+<wire x1="1" y1="-53" x2="1" y2="-56" width="0.1524" layer="91"/>
 <pinref part="GND9" gate="GND" pin="GND"/>
 </segment>
@@
 <wire x1="73" y1="-39" x2="76" y2="-39" width="0.1524" layer="91"/>
 <wire x1="76" y1="-39" x2="76" y2="-17" width="0.1524" layer="91"/>
-<label x="77" y="-16" size="1" layer="95" ratio="12"/>
+<label x="77" y="-17" size="1" layer="95" ratio="12"/>
 <wire x1="76" y1="-17" x2="76" y2="-15" width="0.1524" layer="91"/>
 <wire x1="76" y1="-17" x2="108" y2="-17" width="0.1524" layer="91"/>
@@
 <wire x1="102" y1="-68" x2="102" y2="-104" width="0.1524" layer="91"/>
 <wire x1="102" y1="-104" x2="77" y2="-104" width="0.1524" layer="91"/>
-<label x="23" y="-40" size="1" layer="95" ratio="12"/>
+<label x="-14" y="-40" size="1" layer="95" ratio="12"/>
 <label x="80" y="-104" size="1" layer="95" ratio="12"/>
 <wire x1="22" y1="-68" x2="22" y2="-40" width="0.1524" layer="91"/>
 <pinref part="C4" gate="G$1" pin="1"/>
-<wire x1="-1" y1="-43" x2="-1" y2="-40" width="0.1524" layer="91"/>
+<wire x1="1" y1="-43" x2="1" y2="-40" width="0.1524" layer="91"/>
 <pinref part="R5" gate="G$1" pin="1"/>
-<wire x1="-1" y1="-40" x2="-15" y2="-40" width="0.1524" layer="91"/>
+<wire x1="1" y1="-40" x2="-15" y2="-40" width="0.1524" layer="91"/>
 <pinref part="TP10" gate="G$1" pin="1"/>
 <wire x1="-15" y1="-40" x2="-15" y2="-42" width="0.1524" layer="91"/>
-<wire x1="-1" y1="-40" x2="5" y2="-40" width="0.1524" layer="91"/>
-<junction x="-1" y="-40"/>
-<wire x1="5" y1="-40" x2="22" y2="-40" width="0.1524" layer="91"/>
-<junction x="5" y="-40"/>
+<wire x1="1" y1="-40" x2="7" y2="-40" width="0.1524" layer="91"/>
+<junction x="1" y="-40"/>
+<wire x1="7" y1="-40" x2="22" y2="-40" width="0.1524" layer="91"/>
+<junction x="7" y="-40"/>
 <junction x="22" y="-40"/>
 <pinref part="X1" gate="G$1" pin="3"/>
